File: sepic_charger/sepic_charger.kicad_pcb (KiCad board)
At the start: 2 copper layers, 32 x 18 mm, 27 parts, among them J101 Conn_01x02_Male, J102 Conn_01x02_Male, J104 Conn_01x02_Male, J105 Conn_01x02_Male, J106 Conn_01x02_Male, Q101 NVTFS5C673NLTAG, U101 INA138, U102 UCC2751x

Commit message: Updated design
Parts:
- added C1: 0.1u, Capacitor_SMD:C_0603_1608Metric, F.Cu at (161.8, 101.6)
- added R1: 100k, Resistor_SMD:R_0603_1608Metric, F.Cu at (161.8, 98.6)
- added R2: 22k, Resistor_SMD:R_0603_1608Metric, F.Cu at (161.8, 100.0)
- J105: value Conn_01x02_Male -> Conn_01x03_Male; footprint Connector_PinHeader_2.54mm:PinHeader_1x02_P2.54mm_Vertical -> Connector_PinHeader_2.54mm:PinHeader_1x03_P2.54mm_Vertical
- U101, U102: footprint Package_TO_SOT_SMD:SOT-23-5 -> sot:SOT-23-5
- moved J105 5.68 mm to (164.7, 104.0), turned to 180 degrees
- moved C106 5.15 mm to (157.5, 106.0)
- moved J106 3.21 mm to (164.7, 106.7)
- moved R104 0.21 mm to (164.3, 96.9)
- moved C112 0.10 mm to (165.1, 94.5)
- moved C111 0.10 mm to (161.5, 96.9)
- turned C107 to 0 degrees
- turned C108 to 0 degrees
- turned C109 to 0 degrees
- turned C110 to 0 degrees
Connections:
- C112 pad 2: Net-(C112-Pad2) -> /IMEAS
- J105 pad 2: Net-(C112-Pad2) -> /VMEAS
- R104 pad 2: Net-(C112-Pad2) -> /IMEAS
- U101 pad 1: Net-(C112-Pad2) -> /IMEAS
Routing:
- net /VOUT: track 5.85 -> 13.9 mm, vias 0 -> 1
- net GND: track 10.4 -> 16.3 mm, vias 70 -> 75
- net Net-(C112-Pad2): track 5.76 -> 0.00 mm
- net /IMEAS: track 0.00 -> 5.76 mm
- net /VMEAS: track 0.00 -> 4.97 mm
- net +5V: track 30.4 -> 33.0 mm
