File: buck_charger/buck_charger.kicad_pcb (KiCad board)
At the start: 2 copper layers, 32 x 29.5 mm, 54 parts, among them J101 Conn_01x02_Male, J102 Conn_01x02_Male, J103 Conn_01x05, J104 Conn_01x02_Male, J105 Conn_01x03_Male, J106 Conn_01x05, Q101 PMGD280UN,115, Q102 PMGD280UN,115, U101 RT2862, U102 INA138

Commit message: More stuff
Parts:
- added C118: 0.1u, Capacitor_SMD:C_0603_1608Metric, F.Cu at (143.5, 81.5)
- added C119: 0.1u, Capacitor_SMD:C_0603_1608Metric, F.Cu at (140.5, 81.5)
- added C120: 0.1u, Capacitor_SMD:C_0603_1608Metric, F.Cu at (137.5, 81.5)
- added J107: Conn_01x05, Connector_PinHeader_2.54mm:PinHeader_1x05_P2.54mm_Vertical, F.Cu at (136.8, 85.2)
- added R124: 470k, Resistor_SMD:R_0603_1608Metric, F.Cu at (143.5, 83.0)
- added R125: 100k, Resistor_SMD:R_0603_1608Metric, F.Cu at (143.5, 80.0)
- added R126: 470k, Resistor_SMD:R_0603_1608Metric, F.Cu at (140.5, 83.0)
- added R127: 100k, Resistor_SMD:R_0603_1608Metric, F.Cu at (140.5, 80.0)
- added R128: 470k, Resistor_SMD:R_0603_1608Metric, F.Cu at (137.5, 83.0)
- added R129: 100k, Resistor_SMD:R_0603_1608Metric, F.Cu at (137.5, 80.0)
- J105: value Conn_01x03_Male -> Conn_01x02_Male; footprint Connector_PinHeader_2.54mm:PinHeader_1x03_P2.54mm_Vertical -> Connector_PinHeader_2.54mm:PinHeader_1x02_P2.54mm_Vertical
- R109: value 100k -> 470k
- R110: value 18k -> 100k
- R112, R113, R114, R115: value 100 -> 1k
- moved R110 25.3 mm to (146.5, 80.0), turned to 0 degrees
- moved R109 23.6 mm to (146.5, 83.0), turned to 180 degrees
- moved C109 23.3 mm to (146.5, 81.5), turned to 0 degrees
- moved J103 18.5 mm to (155.9, 88.5)
- moved J106 18.0 mm to (136.9, 88.5)
Connections:
- C109 pad 2: /VMEAS -> /VCELL4
- R109 pad 1: /VMEAS -> /VCELL4
- R109 pad 2: /VOUT -> /CELL4
- R110 pad 2: /VMEAS -> /VCELL4
Routing:
- net /CELL4: track 0.00 -> 31.5 mm, vias 0 -> 2
- net /CELL2: track 8.94 -> 33.3 mm
- net /CELL3: track 11.6 -> 33.6 mm, vias 2 -> 4
- net /CELL1: track 12.5 -> 31.0 mm
- net /DRIVE2: track 0.00 -> 18.4 mm, vias 0 -> 2
- net /DRIVE1: track 0.00 -> 11.7 mm, vias 0 -> 1
- net GND: track 21.5 -> 31.6 mm, vias 63 -> 105
- net /DRIVE4: track 0.00 -> 9.72 mm
- net /CELL3_G: track 1.50 -> 10.4 mm, vias 0 -> 3
- net /VOUT: track 17.4 -> 8.71 mm, vias 2 -> 0
- net /VMEAS: track 6.84 -> 0.00 mm
- net /VCELL1: track 0.00 -> 5.62 mm
- net /DRIVE3: track 0.00 -> 5.52 mm
- net /VCELL2: track 0.00 -> 5.43 mm
- net /VCELL4: track 0.00 -> 5.30 mm
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Other:
- board size 32 x 29.5 mm -> 32 x 37.5 mm
