File: smart_battery.kicad_pcb (KiCad board)
At the start: 2 copper layers, 98 parts, among them J101 Conn_01x02_Male, J102 Conn_01x02_Male, J103 Conn_01x05_Male, J104 Conn_01x02_Male, Q101 SSM3J35AMFV, Q201 PMGD280UN,115, Q202 PMGD280UN,115, U101 NCP716, U102 STM32F051K6Ux, U201 TSV914IPT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

Commit message: Layer, track and mask setup
Other:
- copper layers 2 -> 4
- net class Default: clearance 0.2 -> 0.1; trace_width 0.25 -> 0.1; via_dia 0.8 -> 0.45; via_drill 0.4 -> 0.2
- rule pad_to_mask_clearance: 0.051 -> 0.05
- rule solder_mask_min_width: 0.25 -> 0.09
- rule trace_clearance: 0.2 -> 0.1
- rule trace_min: 0.2 -> 0.1
- rule via_min_drill: 0.3 -> 0.2
- rule via_min_size: 0.4 -> 0.45
Changed lines of the file:
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@@
   (layers
     (0 F.Cu signal)
+    (1 In1.Cu signal)
+    (2 In2.Cu signal)
     (31 B.Cu signal)
     (32 B.Adhes user)
@@
   )
   (setup
-    (last_trace_width 0.25)
-    (trace_clearance 0.2)
+    (last_trace_width 0.1)
+    (trace_clearance 0.1)
     (zone_clearance 0.508)
     (zone_45_only no)
-    (trace_min 0.2)
+    (trace_min 0.1)
     (segment_width 0.2)
     (edge_width 0.15)
-    (via_size 0.8)
-    (via_drill 0.4)
-    (via_min_size 0.4)
-    (via_min_drill 0.3)
+    (via_size 0.45)
+    (via_drill 0.2)
+    (via_min_size 0.45)
+    (via_min_drill 0.2)
     (uvia_size 0.3)
     (uvia_drill 0.1)
@@
     (pad_size 1.524 1.524)
     (pad_drill 0.762)
-    (pad_to_mask_clearance 0.051)
-    (solder_mask_min_width 0.25)
+    (pad_to_mask_clearance 0.05)
+    (solder_mask_min_width 0.09)
     (aux_axis_origin 0 0)
     (visible_elements FFFFFF7F)
@@
   (net 72 "Net-(C103-Pad2)")
   (net_class Default "This is the default net class."
-    (clearance 0.2)
-    (trace_width 0.25)
-    (via_dia 0.8)
-    (via_drill 0.4)
+    (clearance 0.1)
+    (trace_width 0.1)
+    (via_dia 0.45)
+    (via_drill 0.2)
     (uvia_dia 0.3)
     (uvia_drill 0.1)

Commit message: More work
Parts:
- removed U201: TSV914IPT, Package_SO:TSSOP-16_4.4x5mm_P0.65mm
- added C214: 0.1u, passive:C_0402_1005Metric_Rounded, F.Cu at (117.2, 49.2)
- added FB102: BKH1005LM182-T, passive:R_0402_1005Metric_Rounded, F.Cu at (127.1, 46.5)
- added U202: TSV912IQ2T, Package_DFN_QFN:DFN-8-1EP_2x2mm_P0.45mm_EP0.64x1.38mm, F.Cu at (121.1, 47.4)
- added U203: TSV912IQ2T, Package_DFN_QFN:DFN-8-1EP_2x2mm_P0.45mm_EP0.64x1.38mm, F.Cu at (118.0, 47.4)
- FB101: value Ferrite_Bead_Small -> BKH1005LM182-T
Connections:
- D101 pad 2: /BATTERY -> Net-(D101-Pad2)

Commit message: Started PCB layout
Parts:
- removed C104: 0.1u, passive:C_0402_1005Metric_Rounded
- removed R103: 18k, passive:R_0402_1005Metric_Rounded
- removed TH103: 10k, passive:R_0402_1005Metric_Rounded
- D201, D202, Q201, Q202: footprint Package_TO_SOT_SMD:SOT-363_SC-70-6 -> sot:SOT-363
- J101, J102, J104: footprint Connector_PinHeader_2.54mm:PinHeader_1x02_P2.54mm_Vertical -> connectors:1x2_2.54mm
- J103: footprint Connector_PinHeader_2.54mm:PinHeader_1x05_P2.54mm_Vertical -> connectors:1x5_2.54mm
- L301: footprint Inductor_SMD:L_7.3x7.3_H3.5 -> inductor:ASPI-0630LR-HOLE
- Q101: value SSM3J35AMFV -> RZM001P02T2L
- U302: footprint Package_TO_SOT_SMD:SOT-23-6 -> sot:SOT-23-6
- moved J103 85.4 mm to (148.5, 91.5)
- moved J101 78.2 mm to (148.5, 94.0), turned to 180 degrees
- moved C110 65.1 mm to (126.5, 93.5)
- moved U102 65.1 mm to (122.5, 91.0)
- moved C101 64.1 mm to (121.8, 95.2), turned to 90 degrees
- moved R212 64.1 mm to (143.0, 94.0)
- moved TH101 62.9 mm to (138.0, 88.0)
- moved C103 62.6 mm to (132.0, 90.5), turned to 180 degrees
- moved R102 62.6 mm to (123.4, 95.2), turned to 270 degrees
- moved D101 62.4 mm to (132.0, 88.0)
- moved C105 62.3 mm to (128.4, 91.0), turned to 180 degrees
- moved C207 61.3 mm to (138.0, 94.0)
- moved C108 61.2 mm to (118.0, 92.2)
- moved C111 60.4 mm to (118.0, 93.0), turned to 180 degrees
- moved R204 59.6 mm to (135.5, 94.8), turned to 180 degrees
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Connections:
- net Net-(C108-Pad2) renamed /RST
- net Net-(R106-Pad1) renamed /BOOT0
- net Net-(R109-Pad1) renamed /LED1
- net Net-(R110-Pad1) renamed /LED2
- net Net-(R111-Pad1) renamed /LED3
- net Net-(R112-Pad1) renamed /LED4
- net Net-(U102-Pad23) renamed /SWDIO
- U102 pad 15: /TEMP3 -> Net-(U102-Pad15)
- U102 pad 22: Net-(U102-Pad22) -> /AMPS_ONOFF
- U102 pad 24: /AMPS_ONOFF -> /SWCLK
Routing:
- net /buck_charger/CHG_OUT: track 0.00 -> 17.8 mm
- net /VCELL4: track 0.00 -> 1.46 mm
- net /VCELL1: track 0.00 -> 1.45 mm
- net /VCELL3: track 0.00 -> 1.45 mm
- net /VCELL2: track 0.00 -> 1.40 mm
- added copper zone on F.Cu, net /buck_charger/CHG_OUT
- added copper zone on F.Cu, net /buck_charger/SW
- added copper zone on F.Cu, net GND
Other:
- board outline added: 50 x 18 mm

Commit message: More layout and fixes
Parts:
- removed C307: 0.1u, passive:C_0402_1005Metric_Rounded
- removed R307: 50m, Resistor_SMD:R_1206_3216Metric
- removed U302: INA181, sot:SOT-23-6
- added C104: 0.1u, passive:C_0402_1005Metric_Rounded, F.Cu at (133.0, 93.9)
- added R103: 50m, Resistor_SMD:R_1206_3216Metric, F.Cu at (143.0, 96.5)
- added U103: INA181, sot:SOT-23-6, F.Cu at (130.5, 94.4)
- J104: value Conn_01x02_Male -> Dronecode_Debug; footprint connectors:1x2_2.54mm -> connectors:jst-sh-hor-6; moved to B.Cu
- moved FB101 21.9 mm to (124.8, 82.9)
- moved J104 21.2 mm to (120.1, 83.3)
- moved R105 12.3 mm to (120.2, 95.2)
- moved C106 12.1 mm to (121.0, 95.2)
- moved R104 12.0 mm to (119.0, 95.6), turned to 180 degrees
- moved FB102 9.22 mm to (135.5, 88.0)
- moved D103 7.50 mm to (125.0, 81.0)
- moved D105 7.50 mm to (117.0, 81.0)
- moved R107 3.66 mm to (125.8, 86.3), turned to 180 degrees
- moved C301 3.54 mm to (102.9, 94.8), turned to 0 degrees
- moved R108 2.56 mm to (125.8, 85.5), turned to 0 degrees
- moved R110 1.60 mm to (118.9, 82.8)
- moved R112 1.60 mm to (117.3, 82.8)
- moved D102 1.00 mm to (113.0, 81.0)
- moved C212 0.80 mm to (127.9, 82.8)
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Connections:
- net /buck_charger/CHG_OUT renamed /buck_charger/OUT_CHARGER
- C301 pad 1: GND -> GNDPWR
- C302 pad 1: GND -> GNDPWR
- C305 pad 1: GND -> GNDPWR
- C306 pad 1: GND -> GNDPWR
- FB102 pad 2: /BATTERY -> /CELL2
- J101 pad 1: GND -> GNDPWR
- J102 pad 1: GND -> GNDPWR
- J104 pad 1: /RX -> /RST
- R110 pad 1: /LED2 -> /LED4
- R112 pad 1: /LED4 -> /LED2
- R301 pad 1: GND -> GNDPWR
- R302 pad 2: GND -> GNDPWR
- R303 pad 2: GND -> GNDPWR
- R306 pad 1: GND -> GNDPWR
- U102 pad 12: /I_CHG -> /TEMP1
- U102 pad 13: /TEMP1 -> /TEMP2
- U102 pad 14: /TEMP2 -> /I_CHG
- U102 pad 16: /LED1 -> Net-(U102-Pad16)
- U102 pad 26: /LED2 -> /LED4
- U102 pad 28: /LED4 -> /LED2
- U102 pad 32: Net-(U102-Pad32) -> /LED1
- U102 pad 6: /VCELL1 -> /VCELL4
- U102 pad 7: /VCELL2 -> /VCELL3
- U102 pad 8: /VCELL3 -> /VCELL2
- U102 pad 9: /VCELL4 -> /VCELL1
- U202 pad 9: (no net) -> GND
- U203 pad 9: (no net) -> GND
- U301 pad 4: GND -> GNDPWR
- U301 pad 9: GND -> GNDPWR
Routing:
- net /CELL1: track 0.00 -> 45.1 mm, vias 0 -> 6
- net /TEMP2: track 0.00 -> 42.8 mm, vias 0 -> 2
- net GND: track 0.00 -> 41.9 mm, vias 0 -> 77
- net /CELL2: track 0.00 -> 41.3 mm, vias 0 -> 3
- net /AMP_PWR: track 0.00 -> 38.9 mm, vias 0 -> 5
- net /VSET: track 0.00 -> 29.0 mm, vias 0 -> 2
- net /CELL4: track 0.00 -> 27.6 mm, vias 0 -> 1
- net /DCDC_ENABLE: track 0.00 -> 27.5 mm, vias 0 -> 2
- net /CELL3: track 0.00 -> 26.1 mm, vias 0 -> 4
- net +3.3VA: track 0.00 -> 23.8 mm, vias 0 -> 2
- net /VIN_CHG: track 0.00 -> 22.6 mm, vias 0 -> 2
- net /TEMP1: track 0.00 -> 20.7 mm, vias 0 -> 2
- net /VCELL1: track 1.45 -> 21.6 mm, vias 0 -> 2
- net /BAL4: track 0.00 -> 19.1 mm
- net /VCELL3: track 1.45 -> 20.4 mm, vias 0 -> 2
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- added copper zone on F.Cu, net +3V3
- added copper zone on In2.Cu, net +3V3
- added copper zone on F.Cu, net /BATTERY
- added copper zone on B.Cu, net /VIN_CHG
- added copper zone on F.Cu, net /VIN_CHG
- added copper zone on B.Cu, net /buck_charger/OUT_CHARGER
- added copper zone on B.Cu, net GND
- added copper zone on In1.Cu, net GND
- added copper zone on In2.Cu, net GND
- added copper zone on B.Cu, net GNDPWR
- added copper zone on F.Cu, net GNDPWR
- added copper zone on In1.Cu, net GNDPWR
- added copper zone on In2.Cu, net GNDPWR
Other:
- net class Default: clearance 0.1 -> 0.15; trace_width 0.1 -> 0.15
- net class Heat Via added: clearance 0.15, trace_width 0.15, via_dia 0.8, via_drill 0.4
- rule trace_clearance: 0.1 -> 0.15
